File: pcb/GCA.kicad_pcb (KiCad board)
At the start: 2 copper layers, 28.4 x 17 mm, 18 parts, among them J2 Conn_01x05_Pin, SW2 SW_SPDT, U1 AT24CM02-SSHM

Commit message: Flip connector to top
Parts:
- J2: moved to F.Cu
- moved J2 10.2 mm to (116.8, 88.6)
Connections:
- J2 pad 1: VCC -> TWI_E
- J2 pad 2: GND -> SDA
- J2 pad 4: SDA -> GND
- J2 pad 5: TWI_E -> VCC
