File: pcb/GCA.kicad_sch (KiCad schematic)
At the start: 18 parts, among them J2 Conn_01x05_Pin, SW2 SW_SPDT, U1 AT24CM02-SSHM

Commit message: Rename/Add/Remove bom fields
Parts:
- C1: HTL (none) -> 100140; Vendor HTL -> (none); VendorId 100140 -> (none); now in the parts list
- C2: HTL (none) -> 100128; Vendor HTL -> (none); VendorId 100128 -> (none); now in the parts list
- H1: now in the parts list
- J2: HTL (none) -> 101522
- R1, R2, R3, R6: HTL (none) -> 102967; Vendor HTL -> (none); VendorId 102967 -> (none)
- R4, R5: HTL (none) -> 102959; Vendor HTL -> (none); VendorId 102959 -> (none)
- SW2: HTL (none) -> 103603
- U1: HTL (none) -> 103616; Vendor HTL -> (none); VendorId 103616 -> (none)
Changed lines of the file:
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@@
-			)
-		)
-		(property "Vendor" ""
-			(at 242.57 144.78 0)
-			(effects
-				(font
-					(size 1.27 1.27)
-				)
-				(hide yes)
-			)
-		)
-		(property "VendorId" ""
-			(at 242.57 144.78 0)
-			(effects
-				(font
-					(size 1.27 1.27)
-				)
-				(hide yes)
 			)
 		)
@@
 		(unit 1)
 		(exclude_from_sim no)
-		(in_bom no)
+		(in_bom yes)
 		(on_board yes)
 		(dnp no)
@@
 			)
 		)
-		(property "Vendor" "HTL"
-			(at 100.33 88.9 0)
-			(effects
-				(font
-					(size 1.27 1.27)
-				)
-				(hide yes)
-			)
-		)
-		(property "VendorId" "100128"
+		(property "HTL" "100128"
 			(at 100.33 88.9 0)
 			(effects
@@
 			)
 		)
-		(property "Vendor" "HTL"
-			(at 165.1 81.28 0)
-			(effects
-				(font
-					(size 1.27 1.27)
-				)
-				(hide yes)
-			)
-		)
-		(property "VendorId" "102959"
+		(property "HTL" "102959"
 			(at 165.1 81.28 0)
 			(effects
@@
 			)
 		)
-		(property "Vendor" "HTL"
-			(at 193.04 83.82 0)
-			(effects
-				(font
-					(size 1.27 1.27)
-				)
-				(hide yes)
-			)
-		)
-		(property "VendorId" "102967"
+		(property "HTL" "102967"
 			(at 193.04 83.82 0)
 			(effects
@@
 		(unit 1)
 		(exclude_from_sim no)
-		(in_bom no)
+		(in_bom yes)
 		(on_board yes)
 		(dnp no)
@@
 			)
 		)
-		(property "Vendor" "HTL"
-			(at 223.52 90.17 0)
-			(effects
-				(font
-					(size 1.27 1.27)
-				)
-				(hide yes)
-			)
-		)
-		(property "VendorId" "102967"
+		(property "HTL" "102967"
 			(at 223.52 90.17 0)
 			(effects
@@
 			)
 		)
-		(property "Vendor" "HTL"
-			(at 196.85 83.82 0)
-			(effects
-				(font
-					(size 1.27 1.27)
-				)
-				(hide yes)
-			)
-		)
-		(property "VendorId" "102967"
+		(property "HTL" "102967"
 			(at 196.85 83.82 0)
 			(effects
@@
 			)
 		)
-		(property "Vendor" "HTL"
-			(at 161.29 81.28 0)
-			(effects
-				(font
-					(size 1.27 1.27)
-				)
-				(hide yes)
-			)
-		)
-		(property "VendorId" "102959"
+		(property "HTL" "102959"
 			(at 161.29 81.28 0)
 			(effects
@@
 			)
 		)
-		(property "Vendor" "HTL"
-			(at 139.7 83.82 0)
-			(effects
-				(font
-					(size 1.27 1.27)
-				)
-				(hide yes)
-			)
-		)
-		(property "VendorId" "102967"
+		(property "HTL" "102967"
 			(at 139.7 83.82 0)
 			(effects
@@
 		(unit 1)
 		(exclude_from_sim no)
-		(in_bom no)
+		(in_bom yes)
 		(on_board yes)
 		(dnp no)
@@
 			)
 		)
-		(property "Vendor" "HTL"
-			(at 87.63 88.9 0)
-			(effects
-				(font
-					(size 1.27 1.27)
-				)
-				(hide yes)
-			)
-		)
-		(property "VendorId" "100140"
+		(property "HTL" "100140"
 			(at 87.63 88.9 0)
 			(effects
@@
 			)
 		)
-		(property "Vendor" ""
-			(at 229.87 144.78 0)
-			(effects
-				(font
-					(size 1.27 1.27)
-				)
-				(hide yes)
-			)
-		)
-		(property "VendorId" ""
-			(at 229.87 144.78 0)
-			(effects
-				(font
-					(size 1.27 1.27)
-				)
-				(hide yes)
-			)
-		)
 		(instances
 			(project "GCA"
@@
 					(size 1.27 1.27)
 				)
-			)
-		)
-		(property "Vendor" ""
-			(at 204.47 144.78 0)
-			(effects
-				(font
-					(size 1.27 1.27)
-				)
-				(hide yes)
-			)
-		)
-		(property "VendorId" ""
-			(at 204.47 144.78 0)
-			(effects
-				(font
-					(size 1.27 1.27)
-				)
-				(hide yes)
 			)
 		)
@@
 			)
 		)
+		(property "HTL" "101522"
+			(at 69.85 87.63 90)
+			(effects
+				(font
+					(size 1.27 1.27)
+				)
+				(hide yes)
+			)
+		)
 		(pin "2"
 		)
@@
 					(size 1.27 1.27)
 				)
-			)
-		)
-		(property "Vendor" ""
-			(at 217.17 144.78 0)
-			(effects
-				(font
-					(size 1.27 1.27)
-				)
-				(hide yes)
-			)
-		)
-		(property "VendorId" ""
-			(at 217.17 144.78 0)
-			(effects
-				(font
-					(size 1.27 1.27)
-				)
-				(hide yes)
 			)
 		)
@@
 			)
 		)
-		(property "Vendor" "HTL"
-			(at 177.8 88.9 0)
-			(effects
-				(font
-					(size 1.27 1.27)
-				)
-				(hide yes)
-			)
-		)
-		(property "VendorId" "103616"
+		(property "HTL" "103616"
 			(at 177.8 88.9 0)
 			(effects
@@
 			(at 146.05 91.44 0)
 			(effects
+				(font
+					(size 1.27 1.27)
+				)
+				(hide yes)
+			)
+		)
+		(property "HTL" "103603"
+			(at 146.05 91.44 0)
+			(effects
